File: EAGLE Files/Retro Audio Rev2.1.brd (EAGLE design)
At the start: 84 x 70 mm, 72 parts, among them IC1 MAX98357A, Q1 2.5A/30V, Q2 MBT3904DW1T1, Q3 AOD417, SW1 OS102011MA1Q, SW5 PEC11, U2 ESP-WROOM-32, U3 AP2112K-3.3V, U4 FT231XS, X2 19269

Commit message: Updated to show unused parts
Parts:
- C1: value \!0.01uF -> 0.01uF
- R12, R15: value \!300k -> 300k
Changed lines of the file:
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@@
 </attributes>
 <variantdefs>
+<variantdef name="Standard" current="yes"/>
 </variantdefs>
 <classes>
@@
 <attribute name="VALUE" x="79.555" y="23.445" size="0.4064" layer="27" font="vector" ratio="10" rot="R180"/>
 </element>
-<element name="C1" library="microbuilder" package="0603-NO" value="\!0.01uF" x="65.4" y="23.8" smashed="yes" rot="R180">
+<element name="C1" library="microbuilder" package="0603-NO" value="0.01uF" x="65.4" y="23.8" populate="no" smashed="yes" rot="R180">
 <attribute name="VALUE" x="63.622" y="24.562" size="0.4064" layer="27" font="vector" ratio="10" rot="R180"/>
 </element>
@@
 <attribute name="VALUE" x="65.032" y="16.711" size="1.27" layer="27" rot="R90"/>
 </element>
-<element name="R12" library="adafruit" package="R0603" value="\!300k" x="60.8" y="14.8" smashed="yes">
+<element name="R12" library="adafruit" package="R0603" value="300k" x="60.8" y="14.8" populate="no" smashed="yes">
 <attribute name="VALUE" x="59.911" y="12.768" size="1.27" layer="27"/>
 </element>
-<element name="R15" library="adafruit" package="R0603" value="\!300k" x="60.8" y="13.4" smashed="yes" rot="R180">
+<element name="R15" library="adafruit" package="R0603" value="300k" x="60.8" y="13.4" populate="no" smashed="yes" rot="R180">
 <attribute name="VALUE" x="61.689" y="15.432" size="1.27" layer="27" rot="R180"/>
 </element>
